File: circuit/midiclock.sch (KiCad schematic (older format))
At the start: 25 parts

Commit message: MOD: finishing schematics file MOD: adding more documentation
Parts:
- added D1: TAPLED, symbol Device:LED
- added J1: MIDI IN, symbol Connector:DIN-5_180degree
- added J1B1: MIDI Conn, symbol Connector:Conn_01x04_Female
- added J2: MIDI OUT, symbol Connector:DIN-5_180degree
- added J3: 9V, symbol Connector:Jack-DC
- added J3B1: TAP Switch, symbol Connector:Conn_01x02_Female
- added J3B1: Power, symbol Connector:Conn_01x03_Female
- added J4B1: Encoder Board, symbol Connector:Conn_01x05_Female
- added J5: SWITCH 1, Jack-Mono, symbol jack:Jack-Mono
- added J5A1: SWITCHES, symbol Connector:Conn_01x04_Male
- added J5B1: SWITCHES, symbol Connector:Conn_01x04_Female
- added J6: SWITCH 2, Jack-Mono, symbol jack:Jack-Mono
- added R10, R11: 4.7k, symbol Device:R
- added SW1: ENCODER, symbol Device:Rotary_Encoder_Switch
- added SW2: Footswitch, symbol Switch:SW_Push
- added U4, U5: AQY211EH, symbol aqy21:AQY21
- J1A1: renamed from J?; value Conn_01x04_Male -> MIDI
- SW3: renamed from SW?; symbol Switch:SW_Push_Dual -> Switch:SW_Push
- gave numbers to parts that had none: 13
- renumbered R2 to R4, R4 to R5, R3 to R6, R5 to R7
Connections:
- net GND: now also J4.2 (Pin_2), U4.2 (c), U5.2 (c); no longer J4.1 (Pin_1), SW3.4
- net at U3.20 (A3): now also R11.1
- net at C5.1, R3.1, R4.1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: now also J4.1 (Pin_1); no longer J4.2 (Pin_2)
- net at SW3.1, U3.22 (RST): no longer SW3.3
- new net: R10.2, U4.1 (a)
- new net: R11.2, U5.1 (a)
- new net: J5.S (SLEEVE), J5B1.4 (Pin_4)
- new net: J5.T (TIP), J5B1.3 (Pin_3)
- new net: J5B1.2 (Pin_2), J6.S (SLEEVE)
- new net: J5B1.1 (Pin_1), J6.T (TIP)
- new net: J5A1.2 (Pin_2), U4.3 (s1)
- new net: J5A1.1 (Pin_1), U4.4 (s2)
- new net: J5A1.4 (Pin_4), U5.3 (s1)
- new net: J5A1.3 (Pin_3), U5.4 (s2)
- new net: J1.4, J1B1.1 (Pin_1)
- new net: J1.5, J1B1.2 (Pin_2)
- new net: J1B1.3 (Pin_3), J2.4
- new net: J1B1.4 (Pin_4), J2.5
- new net: J3B1.2 (Pin_2), SW2.1
- new net: J3B1.1 (Pin_1), SW2.2
- new net: J4B1.1 (Pin_1), SW1.A
- new net: J4B1.2 (Pin_2), SW1.B
- new net: D1.1 (K), J4B1.5 (Pin_5), SW1.C, SW1.S1
- new net: J4B1.3 (Pin_3), SW1.S2
- new net: D1.2 (A), J4B1.4 (Pin_4)
- new net: J3.1, J3B1.2 (Pin_2)
- new net: J3.2, J3B1.1 (Pin_1), J3B1.3 (Pin_3)
Other:
- moved on the sheet: C1, C2, C3, C4, C5, D2, J1A1, J3A1, J4, J4A1, L1, R1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
